Commit message: Total revolution! Gigantic refactor

File: yumi_description/urdf/yumi.urdf.xacro (robot description, xacro)
@@ -9,7 +9,10 @@
   <!--Import the yumi servo gripper macro -->
   <xacro:include filename="$(find yumi_description)/urdf/Grippers/yumi_servo_gripper.xacro"/>
+  <!--Import the Schunk Mini40 F/T sensor -->
+  <xacro:include filename="$(find yumi_description)/urdf/Sensors/ftsensor.xacro"/>
   <!-- Import Gazebo plugins -->
   <xacro:include filename="$(find yumi_description)/urdf/Gazebo/gazebo.urdf.xacro"/>
   <xacro:property name="yumi_setup" value="$(arg yumi_setup)" />
+  <xacro:property name="yumi_parent" value=" " />
   <xacro:if value="${yumi_setup == 'robot_centric'}">
   	<!-- Pure YuMi URDF, with no joints connecting it to any other robot or pedestal. Neither accessories. -->
@@ -28,11 +31,19 @@
     <origin xyz="0 0 0.1" rpy="0 0 0" />
   </xacro:yumi>
+  <!--right sensor-->
+  <xacro:schunk_mini40 name="ftsensor_r" parent="yumi_link_7_r">
+    <origin xyz="0 0 0.0284" rpy="0 0 ${PI/2}" />
+  </xacro:schunk_mini40>
   <!--right gripper-->
-  <xacro:yumi_servo_gripper name="gripper_r" hardware_interface="hardware_interface/$(arg grippers_interface)" parent="yumi_link_7_r">
-    <origin xyz="0 0 0.007" rpy="0 0 ${PI}" />
+  <xacro:yumi_servo_gripper name="gripper_r" hardware_interface="hardware_interface/$(arg grippers_interface)" parent="ftsensor_r">
+    <origin xyz="0 0 0.004" rpy="0 0 ${PI/2}" />
   </xacro:yumi_servo_gripper>
+  <!--left sensor-->
+  <xacro:schunk_mini40 name="ftsensor_l" parent="yumi_link_7_l">
+    <origin xyz="0 0 0.0284" rpy="0 0 ${PI/2}" />
+  </xacro:schunk_mini40>
   <!--left gripper-->
-  <xacro:yumi_servo_gripper name="gripper_l" hardware_interface="hardware_interface/$(arg grippers_interface)" parent="yumi_link_7_l">
-    <origin xyz="0 0 0.007" rpy="0 0 ${PI}" />
+  <xacro:yumi_servo_gripper name="gripper_l" hardware_interface="hardware_interface/$(arg grippers_interface)" parent="ftsensor_l">
+    <origin xyz="0 0 0.004" rpy="0 0 ${PI/2}" />
   </xacro:yumi_servo_gripper>
 </robot>

File: yumi_description/urdf/yumi.xacro (robot description, xacro)
@@ -24,5 +24,5 @@
         <origin xyz="0 0 0" rpy="0 0 0"/>
         <geometry>
-          <mesh filename="package://yumi_description/meshes/body.stl"/>
+          <mesh filename="package://yumi_description/meshes/yumi/body.stl"/>
         </geometry>
         <material name="Light_Grey"/>
@@ -31,5 +31,5 @@
         <origin xyz="0 0 0" rpy="0 0 0"/>
         <geometry>
-          <mesh filename="package://yumi_description/meshes/coarse/body.stl"/>
+          <mesh filename="package://yumi_description/meshes/yumi/coarse/body.stl"/>
         </geometry>
         <material name="Light_Grey"/>
@@ -56,12 +56,12 @@
         <origin xyz="0 0 0" rpy="0 0 0"/>
         <geometry>
-          <mesh filename="package://yumi_description/meshes/link_1.stl"/>
-        </geometry>
-        <material name="Grey"/>
-      </visual>
-      <collision>
-        <origin xyz="0 0 0" rpy="0 0 0"/>
-        <geometry>
-          <mesh filename="package://yumi_description/meshes/coarse/link_1.stl"/>
+          <mesh filename="package://yumi_description/meshes/yumi/link_1.stl"/>
+        </geometry>
+        <material name="Grey"/>
+      </visual>
+      <collision>
+        <origin xyz="0 0 0" rpy="0 0 0"/>
+        <geometry>
+          <mesh filename="package://yumi_description/meshes/yumi/coarse/link_1.stl"/>
         </geometry>
         <material name="Grey"/>
@@ -87,12 +87,12 @@
         <origin xyz="0 0 0" rpy="0 0 0"/>
         <geometry>
-          <mesh filename="package://yumi_description/meshes/link_2.stl"/>
-        </geometry>
-        <material name="Grey"/>
-      </visual>
-      <collision>
-        <origin xyz="0 0 0" rpy="0 0 0"/>
-        <geometry>
-          <mesh filename="package://yumi_description/meshes/coarse/link_2.stl"/>
+          <mesh filename="package://yumi_description/meshes/yumi/link_2.stl"/>
+        </geometry>
+        <material name="Grey"/>
+      </visual>
+      <collision>
+        <origin xyz="0 0 0" rpy="0 0 0"/>
+        <geometry>
+          <mesh filename="package://yumi_description/meshes/yumi/coarse/link_2.stl"/>
         </geometry>
         <material name="Grey"/>
@@ -118,12 +118,12 @@
         <origin xyz="0 0 0" rpy="0 0 0"/>
         <geometry>
-          <mesh filename="package://yumi_description/meshes/link_3.stl"/>
-        </geometry>
-        <material name="Grey"/>
-      </visual>
-      <collision>
-        <origin xyz="0 0 0" rpy="0 0 0"/>
-        <geometry>
-          <mesh filename="package://yumi_description/meshes/coarse/link_3.stl"/>
+          <mesh filename="package://yumi_description/meshes/yumi/link_3.stl"/>
+        </geometry>
+        <material name="Grey"/>
+      </visual>
+      <collision>
+        <origin xyz="0 0 0" rpy="0 0 0"/>
+        <geometry>
+          <mesh filename="package://yumi_description/meshes/yumi/coarse/link_3.stl"/>
         </geometry>
         <material name="Grey"/>
@@ -149,12 +149,12 @@
         <origin xyz="0 0 0" rpy="0 0 0"/>
         <geometry>
-          <mesh filename="package://yumi_description/meshes/link_4.stl"/>
-        </geometry>
-        <material name="Grey"/>
-      </visual>
-      <collision>
-        <origin xyz="0 0 0" rpy="0 0 0"/>
-        <geometry>
-          <mesh filename="package://yumi_description/meshes/coarse/link_4.stl"/>
+          <mesh filename="package://yumi_description/meshes/yumi/link_4.stl"/>
+        </geometry>
+        <material name="Grey"/>
+      </visual>
+      <collision>
+        <origin xyz="0 0 0" rpy="0 0 0"/>
+        <geometry>
+          <mesh filename="package://yumi_description/meshes/yumi/coarse/link_4.stl"/>
         </geometry>
         <material name="Grey"/>
@@ -180,12 +180,12 @@
         <origin xyz="0 0 0" rpy="0 0 0"/>
         <geometry>
-          <mesh filename="package://yumi_description/meshes/link_5.stl"/>
-        </geometry>
-        <material name="Grey"/>
-      </visual>
-      <collision>
-        <origin xyz="0 0 0" rpy="0 0 0"/>
-        <geometry>
-          <mesh filename="package://yumi_description/meshes/coarse/link_5.stl"/>
+          <mesh filename="package://yumi_description/meshes/yumi/link_5.stl"/>
+        </geometry>
+        <material name="Grey"/>
+      </visual>
+      <collision>
+        <origin xyz="0 0 0" rpy="0 0 0"/>
+        <geometry>
+          <mesh filename="package://yumi_description/meshes/yumi/coarse/link_5.stl"/>
         </geometry>
         <material name="Grey"/>
@@ -211,12 +211,12 @@
         <origin xyz="0 0 0" rpy="0 0 0"/>
         <geometry>
-          <mesh filename="package://yumi_description/meshes/link_6.stl"/>
-        </geometry>
-        <material name="Grey"/>
-      </visual>
-      <collision>
-        <origin xyz="0 0 0" rpy="0 0 0"/>
-        <geometry>
-          <mesh filename="package://yumi_description/meshes/coarse/link_6.stl"/>
+          <mesh filename="package://yumi_description/meshes/yumi/link_6.stl"/>
+        </geometry>
+        <material name="Grey"/>
+      </visual>
+      <collision>
+        <origin xyz="0 0 0" rpy="0 0 0"/>
+        <geometry>
+          <mesh filename="package://yumi_description/meshes/yumi/coarse/link_6.stl"/>
         </geometry>
         <material name="Grey"/>
@@ -242,12 +242,12 @@
         <origin xyz="0 0 0" rpy="0 0 0"/>
         <geometry>
-          <mesh filename="package://yumi_description/meshes/link_7.stl"/>
-        </geometry>
-        <material name="Grey"/>
-      </visual>
-      <collision>
-        <origin xyz="0 0 0" rpy="0 0 0"/>
-        <geometry>
-          <mesh filename="package://yumi_description/meshes/coarse/link_7.stl"/>
+          <mesh filename="package://yumi_description/meshes/yumi/link_7.stl"/>
+        </geometry>
+        <material name="Grey"/>
+      </visual>
+      <collision>
+        <origin xyz="0 0 0" rpy="0 0 0"/>
+        <geometry>
+          <mesh filename="package://yumi_description/meshes/yumi/coarse/link_7.stl"/>
         </geometry>
         <material name="Grey"/>
@@ -274,12 +274,12 @@
         <origin xyz="0 0 0" rpy="0 0 0"/>
         <geometry>
-          <mesh filename="package://yumi_description/meshes/link_1.stl"/>
-        </geometry>
-        <material name="Grey"/>
-      </visual>
-      <collision>
-        <origin xyz="0 0 0" rpy="0 0 0"/>
-        <geometry>
-          <mesh filename="package://yumi_description/meshes/coarse/link_1.stl"/>
+          <mesh filename="package://yumi_description/meshes/yumi/link_1.stl"/>
+        </geometry>
+        <material name="Grey"/>
+      </visual>
+      <collision>
+        <origin xyz="0 0 0" rpy="0 0 0"/>
+        <geometry>
+          <mesh filename="package://yumi_description/meshes/yumi/coarse/link_1.stl"/>
         </geometry>
         <material name="Grey"/>
@@ -305,12 +305,12 @@
         <origin xyz="0 0 0" rpy="0 0 0"/>
         <geometry>
-          <mesh filename="package://yumi_description/meshes/link_2.stl"/>
-        </geometry>
-        <material name="Grey"/>
-      </visual>
-      <collision>
-        <origin xyz="0 0 0" rpy="0 0 0"/>
-        <geometry>
-          <mesh filename="package://yumi_description/meshes/coarse/link_2.stl"/>
+          <mesh filename="package://yumi_description/meshes/yumi/link_2.stl"/>
+        </geometry>
+        <material name="Grey"/>
+      </visual>
+      <collision>
+        <origin xyz="0 0 0" rpy="0 0 0"/>
+        <geometry>
+          <mesh filename="package://yumi_description/meshes/yumi/coarse/link_2.stl"/>
         </geometry>
         <material name="Grey"/>
@@ -336,12 +336,12 @@
         <origin xyz="0 0 0" rpy="0 0 0"/>
         <geometry>
-          <mesh filename="package://yumi_description/meshes/link_3.stl"/>
-        </geometry>
-        <material name="Grey"/>
-      </visual>
-      <collision>
-        <origin xyz="0 0 0" rpy="0 0 0"/>
-        <geometry>
-          <mesh filename="package://yumi_description/meshes/coarse/link_3.stl"/>
+          <mesh filename="package://yumi_description/meshes/yumi/link_3.stl"/>
+        </geometry>
+        <material name="Grey"/>
+      </visual>
+      <collision>
+        <origin xyz="0 0 0" rpy="0 0 0"/>
+        <geometry>
+          <mesh filename="package://yumi_description/meshes/yumi/coarse/link_3.stl"/>
         </geometry>
         <material name="Grey"/>
@@ -367,12 +367,12 @@
         <origin xyz="0 0 0" rpy="0 0 0"/>
         <geometry>
-          <mesh filename="package://yumi_description/meshes/link_4.stl"/>
-        </geometry>
-        <material name="Grey"/>
-      </visual>
-      <collision>
-        <origin xyz="0 0 0" rpy="0 0 0"/>
-        <geometry>
-          <mesh filename="package://yumi_description/meshes/coarse/link_4.stl"/>
+          <mesh filename="package://yumi_description/meshes/yumi/link_4.stl"/>
+        </geometry>
+        <material name="Grey"/>
+      </visual>
+      <collision>
+        <origin xyz="0 0 0" rpy="0 0 0"/>
+        <geometry>
+          <mesh filename="package://yumi_description/meshes/yumi/coarse/link_4.stl"/>
         </geometry>
         <material name="Grey"/>
@@ -398,12 +398,12 @@
         <origin xyz="0 0 0" rpy="0 0 0"/>
         <geometry>
-          <mesh filename="package://yumi_description/meshes/link_5.stl"/>
-        </geometry>
-        <material name="Grey"/>
-      </visual>
-      <collision>
-        <origin xyz="0 0 0" rpy="0 0 0"/>
-        <geometry>
-          <mesh filename="package://yumi_description/meshes/coarse/link_5.stl"/>
+          <mesh filename="package://yumi_description/meshes/yumi/link_5.stl"/>
+        </geometry>
+        <material name="Grey"/>
+      </visual>
+      <collision>
+        <origin xyz="0 0 0" rpy="0 0 0"/>
+        <geometry>
+          <mesh filename="package://yumi_description/meshes/yumi/coarse/link_5.stl"/>
         </geometry>
         <material name="Grey"/>
@@ -429,12 +429,12 @@
         <origin xyz="0 0 0" rpy="0 0 0"/>
         <geometry>
-          <mesh filename="package://yumi_description/meshes/link_6.stl"/>
-        </geometry>
-        <material name="Grey"/>
-      </visual>
-      <collision>
-        <origin xyz="0 0 0" rpy="0 0 0"/>
-        <geometry>
-          <mesh filename="package://yumi_description/meshes/coarse/link_6.stl"/>
+          <mesh filename="package://yumi_description/meshes/yumi/link_6.stl"/>
+        </geometry>
+        <material name="Grey"/>
+      </visual>
+      <collision>
+        <origin xyz="0 0 0" rpy="0 0 0"/>
+        <geometry>
+          <mesh filename="package://yumi_description/meshes/yumi/coarse/link_6.stl"/>
         </geometry>
         <material name="Grey"/>
@@ -460,12 +460,12 @@
         <origin xyz="0 0 0" rpy="0 0 0"/>
         <geometry>
-          <mesh filename="package://yumi_description/meshes/link_7.stl"/>
-        </geometry>
-        <material name="Grey"/>
-      </visual>
-      <collision>
-        <origin xyz="0 0 0" rpy="0 0 0"/>
-        <geometry>
-          <mesh filename="package://yumi_description/meshes/coarse/link_7.stl"/>
+          <mesh filename="package://yumi_description/meshes/yumi/link_7.stl"/>
+        </geometry>
+        <material name="Grey"/>
+      </visual>
+      <collision>
+        <origin xyz="0 0 0" rpy="0 0 0"/>
+        <geometry>
+          <mesh filename="package://yumi_description/meshes/yumi/coarse/link_7.stl"/>
         </geometry>
         <material name="Grey"/>

File: yumi_description/urdf/yumi_ORIGINAL.urdf (robot description, URDF)
Before this commit: robot yumi, 24 links, 23 joints
Links:
- removed link ftsensor_l
- removed link ftsensor_r
Joints:
- removed joint ftsensor_l_joint
- removed joint ftsensor_r_joint
- joint yumi_link_7_l_joint: child ftsensor_l -> gripper_l_base; origin xyz=0 0 0.0284 rpy=0 0 1.57079632679 -> xyz=0 0 0.007 rpy=0 0 3.14159265359
- joint yumi_link_7_r_joint: child ftsensor_r -> gripper_r_base; origin xyz=0 0 0.0284 rpy=0 0 1.57079632679 -> xyz=0 0 0.007 rpy=0 0 3.14159265359

Commit message: Changed package name

File: yumi_description/urdf/yumi.urdf.xacro (robot description, xacro)
@@ -5,7 +5,7 @@
   <!-- Import utilities -->
   <xacro:include filename="$(find yumi_description)/urdf/Util/utilities.xacro" />
-  <!--Import the yumi macro -->
+  <!--Import the yumi xacro -->
   <xacro:include filename="$(find yumi_description)/urdf/yumi.xacro"/>
-  <!--Import the yumi servo gripper macro -->
+  <!--Import the yumi servo gripper xacro -->
   <xacro:include filename="$(find yumi_description)/urdf/Grippers/yumi_servo_gripper.xacro"/>
   <!--Import the Schunk Mini40 F/T sensor -->
@@ -24,5 +24,20 @@
       <parent link="world"/>
       <child link="yumi_base_link"/>
-      <origin xyz="0 0 0.1" rpy="0 0 0" />
+      <!-- <origin xyz="0 0 0.1" rpy="0 0 0" /> -->
+      <origin xyz="0.181 0 0" rpy="0 0 0" />
+    </joint>
+    <!-- right gripper -->
+    <link name="yumi_grip_r"/>
+    <joint name="yumi_grip_r_joint" type="fixed">
+      <parent link="yumi_link_7_r"/>
+      <child link="yumi_grip_r"/>
+      <origin xyz="0 0 0.166" rpy="0 0 0" />
+    </joint>
+    <!-- left gripper -->
+    <link name="yumi_grip_l"/>
+    <joint name="yumi_grip_l_joint" type="fixed">
+      <parent link="yumi_link_7_l"/>
+      <child link="yumi_grip_r"/>
+      <origin xyz="0 0 0.166" rpy="0 0 0" />
     </joint>
   </xacro:if>
