Commit message: Fixed sensor orientation in URDF, changed kinematics update_rate

File: yumi_description/urdf/yumi.urdf (robot description, URDF)
Before this commit: robot yumi, 31 links, 30 joints
Joints:
- joint yumi_link_7_l_joint: origin xyz=0 0 0.007 rpy=0 0 1.57079632679 -> xyz=0 0 0.007 rpy=0 0 0
- joint yumi_link_7_r_joint: origin xyz=0 0 0.007 rpy=0 0 1.57079632679 -> xyz=0 0 0.007 rpy=0 0 0

File: yumi_description/urdf/yumi.urdf.xacro (robot description, xacro)
@@ -24,5 +24,5 @@
   <!--right sensor-->
   <xacro:schunk_mini40 name="ftsensor_r" parent="yumi_link_7_r">
-    <origin xyz="0 0 0.007" rpy="0 0 ${PI/2}" />
+    <origin xyz="0 0 0.007" rpy="0 0 0" />
   </xacro:schunk_mini40>
   <!--right gripper-->
@@ -32,5 +32,5 @@
   <!--left sensor-->
   <xacro:schunk_mini40 name="ftsensor_l" parent="yumi_link_7_l">
-    <origin xyz="0 0 0.007" rpy="0 0 ${PI/2}" />
+    <origin xyz="0 0 0.007" rpy="0 0 0" />
   </xacro:schunk_mini40>
   <!--left gripper-->
