Commit message: Multiple refactors, added simple IK, updated URDF and README WIP trajectory refactoring

File: yumi_description/urdf/Grippers/smart_gripper.gazebo.xacro (robot description, xacro)
@@ -1,5 +1,5 @@
 <?xml version="1.0"?>
-<robot name="yumi_servo_gripper" xmlns:xacro="http://www.ros.org/wiki/xacro">
-  <xacro:macro name="yumi_servo_gripper_gazebo" params="name">
+<robot name="smart_gripper" xmlns:xacro="http://www.ros.org/wiki/xacro">
+  <xacro:macro name="smart_gripper_gazebo" params="name">
   <!-- Plugin for the mimic o/c joint - AFAIK, that shouldn't be necessary any more starting with Gazebo 3.0 -->
     <gazebo>

File: yumi_description/urdf/Grippers/smart_gripper.xacro (robot description, xacro)
@@ -1,15 +1,15 @@
 <?xml version="1.0"?>
 <robot name="yumi" xmlns:xacro="http://www.ros.org/wiki/xacro">
-    <!-- Import all Gazebo-customization elements, including Gazebo colors -->
-    <xacro:include filename="$(find yumi_description)/urdf/Grippers/yumi_servo_gripper.gazebo.xacro" />
-    <!-- Import Transmissions -->
-    <xacro:include filename="$(find yumi_description)/urdf/Grippers/yumi_servo_gripper.transmission.xacro" />
-    <xacro:include filename="$(find hector_xacro_tools)/urdf/inertia_tensors.urdf.xacro" />
-    <!-- some constants -->
-    <xacro:property name="joint_damping" value="0.5" />
-    <xacro:property name="gripper_joint_damping" value="1.0" />
-    <xacro:property name="max_gripper_effort" value="20"/>
-    <xacro:property name="max_gripper_velocity" value="2"/>
-  <xacro:macro name="yumi_servo_gripper" params="parent name hardware_interface *origin">
+  <!-- Import all Gazebo-customization elements, including Gazebo colors -->
+  <xacro:include filename="$(find yumi_description)/urdf/Grippers/smart_gripper.gazebo.xacro" />
+  <!-- Import Transmissions -->
+  <xacro:include filename="$(find yumi_description)/urdf/Grippers/smart_gripper.transmission.xacro" />
+  <xacro:include filename="$(find hector_xacro_tools)/urdf/inertia_tensors.urdf.xacro" />
+  <!-- some constants -->
+  <xacro:property name="joint_damping" value="0.5" />
+  <xacro:property name="gripper_joint_damping" value="1.0" />
+  <xacro:property name="max_gripper_effort" value="20"/>
+  <xacro:property name="max_gripper_velocity" value="2"/>
+  <xacro:macro name="smart_gripper" params="parent name hardware_interface *origin">
     <!--joint between {parent} and base-->
     <joint name="${parent}_joint" type="fixed">
@@ -94,7 +94,14 @@
       </collision>
     </link>
-     <!--Extensions -->
-    <xacro:yumi_servo_gripper_gazebo name="${name}" />
-    <xacro:yumi_servo_gripper_transmission name="${name}" hardware_interface="${hardware_interface}"/>
+    <!-- joint for gripper tip -->
+    <link name="${name}_tip"/>
+    <joint name="${name}_tip_joint" type="fixed">
+      <parent link="${name}_base"/>
+      <child link="${name}_tip"/>
+      <origin xyz="0 0 0.136" rpy="0 0 ${-PI/2}" />
+    </joint>
+     <!-- extensions -->
+    <xacro:smart_gripper_gazebo name="${name}" />
+    <xacro:smart_gripper_transmission name="${name}" hardware_interface="${hardware_interface}"/>
   </xacro:macro>
 </robot>

File: yumi_description/urdf/Sensors/ftsensor.xacro (robot description, xacro)
@@ -32,5 +32,5 @@
     </link>
      <!--Extensions -->
-    <xacro:yumi_servo_gripper_gazebo name="${name}" />
+    <xacro:schunk_mini40_gazebo name="${name}" />
   </xacro:macro>
 </robot>

File: yumi_description/urdf/yumi.urdf (robot description, URDF)
Before this commit: robot yumi, 24 links, 23 joints
Links:
- added link gripper_l_tip
- added link gripper_r_tip
Joints:
- added joint gripper_l_tip_joint: type fixed, parent gripper_l_base, child gripper_l_tip, origin xyz=0 0 0.136 rpy=0 0 -1.57079632679
- added joint gripper_r_tip_joint: type fixed, parent gripper_r_base, child gripper_r_tip, origin xyz=0 0 0.136 rpy=0 0 -1.57079632679
- joint ftsensor_l_joint: origin xyz=0 0 0.004 rpy=0 0 1.57079632679 -> xyz=0 0 0.008 rpy=0 0 1.57079632679
- joint ftsensor_r_joint: origin xyz=0 0 0.004 rpy=0 0 1.57079632679 -> xyz=0 0 0.008 rpy=0 0 1.57079632679
- joint yumi_link_7_l_joint: origin xyz=0 0 0.0284 rpy=0 0 1.57079632679 -> xyz=0 0 0.031 rpy=0 0 1.57079632679
- joint yumi_link_7_r_joint: origin xyz=0 0 0.0284 rpy=0 0 1.57079632679 -> xyz=0 0 0.031 rpy=0 0 1.57079632679

File: yumi_description/urdf/yumi.urdf.xacro (robot description, xacro)
@@ -8,5 +8,5 @@
   <xacro:include filename="$(find yumi_description)/urdf/yumi.xacro"/>
   <!--Import the yumi servo gripper xacro -->
-  <xacro:include filename="$(find yumi_description)/urdf/Grippers/yumi_servo_gripper.xacro"/>
+  <xacro:include filename="$(find yumi_description)/urdf/Grippers/smart_gripper.xacro"/>
   <!--Import the Schunk Mini40 F/T sensor -->
   <xacro:include filename="$(find yumi_description)/urdf/Sensors/ftsensor.xacro"/>
@@ -20,24 +20,10 @@
   <xacro:if value="${yumi_setup == 'default'}">
     <xacro:property name="yumi_parent" value="world" />
+    <!-- world frame -->
     <link name="world"/>
     <joint name="world_joint" type="fixed">
-      <parent link="world"/>
-      <child link="yumi_base_link"/>
-      <!-- <origin xyz="0 0 0.1" rpy="0 0 0" /> -->
-      <origin xyz="0.181 0 0" rpy="0 0 0" />
-    </joint>
-    <!-- right gripper -->
-    <link name="yumi_grip_r"/>
-    <joint name="yumi_grip_r_joint" type="fixed">
-      <parent link="yumi_link_7_r"/>
-      <child link="yumi_grip_r"/>
-      <origin xyz="0 0 0.166" rpy="0 0 0" />
-    </joint>
-    <!-- left gripper -->
-    <link name="yumi_grip_l"/>
-    <joint name="yumi_grip_l_joint" type="fixed">
-      <parent link="yumi_link_7_l"/>
-      <child link="yumi_grip_r"/>
-      <origin xyz="0 0 0.166" rpy="0 0 0" />
+      <parent link="yumi_base_link"/>
+      <child link="world"/>
+      <origin xyz="0.181 0 0" rpy="0 0 ${-PI/2}" />
     </joint>
   </xacro:if>
@@ -48,17 +34,17 @@
   <!--right sensor-->
   <xacro:schunk_mini40 name="ftsensor_r" parent="yumi_link_7_r">
-    <origin xyz="0 0 0.0284" rpy="0 0 ${PI/2}" />
+    <origin xyz="0 0 0.031" rpy="0 0 ${PI/2}" />
   </xacro:schunk_mini40>
   <!--right gripper-->
-  <xacro:yumi_servo_gripper name="gripper_r" hardware_interface="hardware_interface/$(arg grippers_interface)" parent="ftsensor_r">
-    <origin xyz="0 0 0.004" rpy="0 0 ${PI/2}" />
-  </xacro:yumi_servo_gripper>
+  <xacro:smart_gripper name="gripper_r" hardware_interface="hardware_interface/$(arg grippers_interface)" parent="ftsensor_r">
+    <origin xyz="0 0 0.008" rpy="0 0 ${PI/2}" />
+  </xacro:smart_gripper>
   <!--left sensor-->
   <xacro:schunk_mini40 name="ftsensor_l" parent="yumi_link_7_l">
-    <origin xyz="0 0 0.0284" rpy="0 0 ${PI/2}" />
+    <origin xyz="0 0 0.031" rpy="0 0 ${PI/2}" />
   </xacro:schunk_mini40>
   <!--left gripper-->
-  <xacro:yumi_servo_gripper name="gripper_l" hardware_interface="hardware_interface/$(arg grippers_interface)" parent="ftsensor_l">
-    <origin xyz="0 0 0.004" rpy="0 0 ${PI/2}" />
-  </xacro:yumi_servo_gripper>
+  <xacro:smart_gripper name="gripper_l" hardware_interface="hardware_interface/$(arg grippers_interface)" parent="ftsensor_l">
+    <origin xyz="0 0 0.008" rpy="0 0 ${PI/2}" />
+  </xacro:smart_gripper>
 </robot>
