Commit message: Controller class decluttering
Moved "gripper tip" frame from ROS broadcaster in controller to URDF files
WIP completely move kinematics into kdl_kinematics.cpp

File: yumi_description/urdf/Grippers/smart_gripper.xacro (robot description, xacro)
@@ -14,7 +14,7 @@
     <!--joint between {parent} and base-->
     <joint name="${parent}_joint" type="fixed">
-      <xacro:insert_block name="origin"/>
       <parent link="${parent}"/>
       <child link="${name}_base"/>
+      <xacro:insert_block name="origin"/>
     </joint>
     <link name="${name}_base">
@@ -95,10 +95,10 @@
     </link>
     <!-- joint for gripper tip -->
-    <link name="${name}_tip"/>
     <joint name="${name}_tip_joint" type="fixed">
       <parent link="${name}_base"/>
       <child link="${name}_tip"/>
-      <origin xyz="0 0 0.136" rpy="0 0 ${-PI/2}" />
+      <origin xyz="0 0 0.136" rpy="0 0 ${PI}" />
     </joint>
+    <link name="${name}_tip"/>
      <!-- extensions -->
     <xacro:smart_gripper_gazebo name="${name}" />

File: yumi_description/urdf/Sensors/ftsensor.xacro (robot description, xacro)
@@ -6,7 +6,13 @@
     <!--joint between {parent} and base-->
     <joint name="${parent}_joint" type="fixed">
+      <parent link="${parent}"/>
+      <child link="${name}_base"/>
       <xacro:insert_block name="origin"/>
-      <parent link="${parent}"/>
+    </joint>
+    <link name="${name}_base"/>
+    <joint name="${name}_base_joint" type="fixed">
+      <parent link="${name}_base"/>
       <child link="${name}"/>
+      <origin xyz="0 0 ${0.010 + 0.014}" rpy="0 0 ${PI/2}" />
     </joint>
     <link name="${name}">
@@ -31,4 +37,10 @@
       </collision>
     </link>
+    <joint name="${name}_joint" type="fixed">
+      <parent link="${name}"/>
+      <child link="${name}_tool"/>
+      <origin xyz="0 0 0.008" rpy="0 0 0" />
+    </joint>
+    <link name="${name}_tool"/>
      <!--Extensions -->
     <xacro:schunk_mini40_gazebo name="${name}" />

File: yumi_description/urdf/yumi.urdf (robot description, URDF)
Before this commit: robot yumi, 26 links, 25 joints
Links:
- added link ftsensor_l_base
- added link ftsensor_l_tool
- added link ftsensor_r_base
- added link ftsensor_r_tool
Joints:
- added joint ftsensor_l_base_joint: type fixed, parent ftsensor_l_base, child ftsensor_l, origin xyz=0 0 0.024 rpy=0 0 1.57079632679
- added joint ftsensor_l_tool_joint: type fixed, parent ftsensor_l_tool, child gripper_l_base, origin xyz=0 0 0 rpy=0 0 1.57079632679
- added joint ftsensor_r_base_joint: type fixed, parent ftsensor_r_base, child ftsensor_r, origin xyz=0 0 0.024 rpy=0 0 1.57079632679
- added joint ftsensor_r_tool_joint: type fixed, parent ftsensor_r_tool, child gripper_r_base, origin xyz=0 0 0 rpy=0 0 1.57079632679
- joint ftsensor_l_joint: child gripper_l_base -> ftsensor_l_tool; origin xyz=0 0 0.008 rpy=0 0 1.57079632679 -> xyz=0 0 0.008 rpy=0 0 0
- joint ftsensor_r_joint: child gripper_r_base -> ftsensor_r_tool; origin xyz=0 0 0.008 rpy=0 0 1.57079632679 -> xyz=0 0 0.008 rpy=0 0 0
- joint gripper_l_tip_joint: origin xyz=0 0 0.136 rpy=0 0 -1.57079632679 -> xyz=0 0 0.136 rpy=0 0 3.14159265359
- joint gripper_r_tip_joint: origin xyz=0 0 0.136 rpy=0 0 -1.57079632679 -> xyz=0 0 0.136 rpy=0 0 3.14159265359
- joint yumi_link_7_l_joint: child ftsensor_l -> ftsensor_l_base; origin xyz=0 0 0.031 rpy=0 0 1.57079632679 -> xyz=0 0 0.007 rpy=0 0 1.57079632679
- joint yumi_link_7_r_joint: child ftsensor_r -> ftsensor_r_base; origin xyz=0 0 0.031 rpy=0 0 1.57079632679 -> xyz=0 0 0.007 rpy=0 0 1.57079632679

File: yumi_description/urdf/yumi.urdf.xacro (robot description, xacro)
@@ -21,5 +21,4 @@
     <xacro:property name="yumi_parent" value="world" />
     <!-- world frame -->
-    <link name="world"/>
     <joint name="world_joint" type="fixed">
       <parent link="yumi_base_link"/>
@@ -27,4 +26,5 @@
       <origin xyz="0.181 0 0" rpy="0 0 ${-PI/2}" />
     </joint>
+    <link name="world"/>
   </xacro:if>
   <!--yumi-->
@@ -34,17 +34,17 @@
   <!--right sensor-->
   <xacro:schunk_mini40 name="ftsensor_r" parent="yumi_link_7_r">
-    <origin xyz="0 0 0.031" rpy="0 0 ${PI/2}" />
+    <origin xyz="0 0 0.007" rpy="0 0 ${PI/2}" />
   </xacro:schunk_mini40>
   <!--right gripper-->
-  <xacro:smart_gripper name="gripper_r" hardware_interface="hardware_interface/$(arg grippers_interface)" parent="ftsensor_r">
-    <origin xyz="0 0 0.008" rpy="0 0 ${PI/2}" />
+  <xacro:smart_gripper name="gripper_r" hardware_interface="hardware_interface/$(arg grippers_interface)" parent="ftsensor_r_tool">
+    <origin xyz="0 0 0" rpy="0 0 ${PI/2}" />
   </xacro:smart_gripper>
   <!--left sensor-->
   <xacro:schunk_mini40 name="ftsensor_l" parent="yumi_link_7_l">
-    <origin xyz="0 0 0.031" rpy="0 0 ${PI/2}" />
+    <origin xyz="0 0 0.007" rpy="0 0 ${PI/2}" />
   </xacro:schunk_mini40>
   <!--left gripper-->
-  <xacro:smart_gripper name="gripper_l" hardware_interface="hardware_interface/$(arg grippers_interface)" parent="ftsensor_l">
-    <origin xyz="0 0 0.008" rpy="0 0 ${PI/2}" />
+  <xacro:smart_gripper name="gripper_l" hardware_interface="hardware_interface/$(arg grippers_interface)" parent="ftsensor_l_tool">
+    <origin xyz="0 0 0" rpy="0 0 ${PI/2}" />
   </xacro:smart_gripper>
 </robot>
