Commit message: Decluttering and kinematics, WIP demo, found bug
Riorganized yumi URDF, replaced "world" with "workspace"
Completely moved kinematic chains to C++
Sensors now start with modified correct tool tip frame
Renamed "world_tip" topic to simply "world"
Changed name of rViz file
Fixed touchboard demo, found a bug in pose_abs

File: yumi_description/urdf/Yumi/yumi.xacro (robot description, xacro)
@@ -2,14 +2,14 @@
 <robot name="yumi" xmlns:xacro="http://www.ros.org/wiki/xacro">
   <!-- Import all Gazebo-customization elements, including Gazebo colors -->
-  <xacro:include filename="$(find yumi_description)/urdf/Gazebo/yumi.gazebo.xacro" />
+  <xacro:include filename="$(find yumi_description)/urdf/Yumi/yumi.gazebo.xacro" />
   <!-- Import Transmissions -->
-  <xacro:include filename="$(find yumi_description)/urdf/yumi.transmission.xacro" />
+  <xacro:include filename="$(find yumi_description)/urdf/Yumi/yumi.transmission.xacro" />
   <!-- some constants -->
   <xacro:property name="joint_damping" value="0.5" />
   <xacro:property name="max_effort" value="300"/>
-  <xacro:macro name="yumi" params="parent name hardware_interface *origin">
-    <link name="yumi_base_link"></link>
+  <xacro:macro name="yumi" params="name hardware_interface">
+    <link name="${name}_base_link"/>
     <joint name="${name}_base_link_to_body" type="fixed">
-      <parent link="yumi_base_link"/>
+      <parent link="${name}_base_link"/>
       <child link="${name}_body"/>
       <origin xyz="0 0 0" rpy="0 0 0"/>

File: yumi_description/urdf/yumi.urdf (robot description, URDF)
Before this commit: robot yumi, 30 links, 29 joints
Links:
- added link workspace
Joints:
- added joint workspace_joint: type fixed, parent yumi_base_link, child workspace, origin xyz=0.181 0 0 rpy=0 0 -1.57079632679

File: yumi_description/urdf/yumi.urdf.xacro (robot description, xacro)
@@ -5,31 +5,21 @@
   <!-- Import utilities -->
   <xacro:include filename="$(find yumi_description)/urdf/Util/utilities.xacro" />
+  <!-- Import Gazebo plugins -->
+  <xacro:include filename="$(find yumi_description)/urdf/Yumi/gazebo.urdf.xacro"/>
   <!--Import the yumi xacro -->
-  <xacro:include filename="$(find yumi_description)/urdf/yumi.xacro"/>
+  <xacro:include filename="$(find yumi_description)/urdf/Yumi/yumi.xacro"/>
   <!--Import the yumi servo gripper xacro -->
   <xacro:include filename="$(find yumi_description)/urdf/Grippers/smart_gripper.xacro"/>
   <!--Import the Schunk Mini40 F/T sensor -->
   <xacro:include filename="$(find yumi_description)/urdf/Sensors/ftsensor.xacro"/>
-  <!-- Import Gazebo plugins -->
-  <xacro:include filename="$(find yumi_description)/urdf/Gazebo/gazebo.urdf.xacro"/>
-  <xacro:property name="yumi_setup" value="$(arg yumi_setup)" />
-  <xacro:property name="yumi_parent" value=" " />
-  <xacro:if value="${yumi_setup == 'robot_centric'}">
-  	<!-- Pure YuMi URDF, with no joints connecting it to any other robot or pedestal. Neither accessories. -->
-  </xacro:if>
-  <xacro:if value="${yumi_setup == 'default'}">
-    <xacro:property name="yumi_parent" value="world" />
-    <!-- world frame -->
-    <joint name="world_joint" type="fixed">
-      <parent link="yumi_base_link"/>
-      <child link="world"/>
-      <origin xyz="0.181 0 0" rpy="0 0 ${-PI/2}" />
-    </joint>
-    <link name="world"/>
-  </xacro:if>
   <!--yumi-->
-  <xacro:yumi name="yumi" hardware_interface="hardware_interface/$(arg arms_interface)" parent="${yumi_parent}" >
-    <origin xyz="0 0 0.1" rpy="0 0 0" />
-  </xacro:yumi>
+  <xacro:yumi name="yumi" hardware_interface="hardware_interface/$(arg arms_interface)"/>
+  <!-- workspace (i.e. world/task frame) -->
+  <joint name="workspace_joint" type="fixed">
+    <parent link="yumi_base_link"/>
+    <child link="workspace"/>
+    <origin xyz="0.181 0 0" rpy="0 0 ${-PI/2}" />
+  </joint>
+  <link name="workspace"/>
   <!--right sensor-->
   <xacro:schunk_mini40 name="ftsensor_r" parent="yumi_link_7_r">
